Commit message: WIP

File: data/ur5/ur5.urdf (robot description, URDF)
Before this commit: robot ur5, 11 links, 10 joints
Links:
- link base_link: geometry collision mesh filename=collision/base.stl; visual mesh filename=visual/base.dae
- link forearm_link: geometry collision mesh filename=collision/forearm.stl; visual mesh filename=visual/forearm.dae
- link shoulder_link: geometry collision mesh filename=collision/shoulder.stl; visual mesh filename=visual/shoulder.dae
- link upper_arm_link: geometry collision mesh filename=collision/upperarm.stl; visual mesh filename=visual/upperarm.dae
- link wrist_1_link: geometry collision mesh filename=collision/wrist1.stl; visual mesh filename=visual/wrist1.dae
- link wrist_2_link: geometry collision mesh filename=collision/wrist2.stl; visual mesh filename=visual/wrist2.dae
- link wrist_3_link: geometry collision mesh filename=collision/wrist3.stl; visual mesh filename=visual/wrist3.dae
